Commit message: updated

File: torobo_ros/toroboarm_robot/toroboarm_gripper_description/urdf/toroboarm_gripper.urdf.xacro (robot description, xacro)
@@ -6,5 +6,5 @@
   <xacro:include filename="$(find toroboarm_gripper_description)/urdf/sensors/kinect.urdf.xacro"/>
   <!-- =============== Constants =============== -->
-  <property name="M_PI" value="3.1415926535897931"/>
+  <xacro:property name="M_PI" value="3.1415926535897931"/>
   <material name="White">
     <color rgba="1.0 1.0 1.0 1.0"/>

File: torobo_ros/toroboarm_robot/toroboarm_seven_description/urdf/toroboarm.urdf.xacro (robot description, xacro)
@@ -5,5 +5,5 @@
   <xacro:include filename="$(find toroboarm_seven_description)/urdf/toroboarm.transmission.xacro"/>
   <!-- =============== Constants =============== -->
-  <property name="M_PI" value="3.1415926535897931"/>
+  <xacro:property name="M_PI" value="3.1415926535897931"/>
   <!-- =============== Link & Joint =============== -->
   <!-- <link name="base_link"/> -->
